File: tinyAVR-business-card.kicad_sch (KiCad schematic)
At the start: 28 parts, among them J1 Conn_01x12_Female, J2 Conn_01x12_Female, SW1 SW_Push, SW2 SW_Push, SW3 PWR_SEL, U1 ATtiny3227-M, Y1 32.768kHz

Commit message: correct type on tinyAVR 1-series
Other:
- title: tinyAVR 1-Series Business Card -> tinyAVR 2-Series Business Card + Clock + Dev Board
Changed lines of the file:
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@@
   (paper "A4")
   (title_block
-    (title "tinyAVR 1-Series Business Card")
+    (title "tinyAVR 2-Series Business Card + Clock + Dev Board")
     (date "2024-05-10")
     (rev "1.0")
     (company "www.e-tinkers.com")
+    (comment 1 "Hackaday 2024 Business Card Challenge Contest")
     (comment 2 "Designed By: Henry Cheung")
   )
